File: miscellany.kicad_sch (KiCad schematic)
At the start: 12 parts, among them U3 74HC112, U5 74HC123

Commit message: move custom symbols and footprints to project libraries
Parts:
- U3: symbol local:74HC112 -> am9511-6502-symbols:74HC112
- U5: symbol 74xx:74HC123 -> am9511-6502-symbols:74HC123
Other:
- title: (none) -> AM9511 Interface for 6509
Changed lines of the file:
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@@
 	(generator_version "9.0")
 	(paper "USLetter")
+	(title_block
+		(title "AM9511 Interface for 6509")
+	)
 	(junction
 		(at 73.66 124.46)
@@
 	)
 	(symbol
-		(lib_id "local:74HC112")
+		(lib_id "am9511-6502-symbols:74HC112")
 		(at 24.13 182.88 0)
 		(unit 3)
@@
 	)
 	(symbol
-		(lib_id "74xx:74HC123")
+		(lib_id "am9511-6502-symbols:74HC123")
 		(at 48.26 182.88 0)
 		(unit 3)
@@
 	)
 	(symbol
-		(lib_id "74xx:74HC123")
+		(lib_id "am9511-6502-symbols:74HC123")
 		(at 140.97 182.88 0)
 		(unit 2)
